Commit message: created calibration configuration with yaml

File: lemonbot_description/urdf/lemonbot.urdf.xacro (robot description, xacro)
@@ -1,5 +1,8 @@
 <?xml version="1.0"?>
 <robot
-    xmlns:xacro="http://ros.org/wiki/xacro" name="lemonbot">
+    xmlns:xacro="http://www.ros.org/wiki/xacro" name="lemonbot">
+    <xacro:arg name="calibrated" default="false"/>
+    <xacro:arg name="laser_calibration_file" default="$(find lemonbot_calibration)/calibration/camera_calibration.yaml" />
+    <xacro:arg name="camera_calibration_file" default="$(find lemonbot_calibration)/calibration/camera_calibration.yaml" />
     <xacro:include filename="$(find lemonbot_description)/urdf/lemonbot_macro.urdf.xacro"/>
     <xacro:lemonbot prefix="lemonbot" />

File: lemonbot_description/urdf/lemonbot_macro.urdf.xacro (robot description, xacro)
@@ -1,5 +1,8 @@
 <?xml version="1.0"?>
 <robot
-    xmlns:xacro="http://ros.org/wiki/xacro">
+    xmlns:xacro="http://www.ros.org/wiki/xacro">
+    <xacro:arg name="calibrated" default="false"/>
+    <xacro:arg name="laser_calibration_file" default="" />
+    <xacro:arg name="camera_calibration_file" default="" />
     <!-- include all the dependencies -->
     <!-- include asus_camera macro from hector_sensors_description -->
@@ -9,4 +12,13 @@
     <!-- include sick lms1xx macro from lms1xx -->
     <xacro:include filename="$(find lms1xx)/urdf/sick_lms1xx.urdf.xacro" />
+    <!-- load calibration -->
+    <xacro:unless value="$(arg calibrated)">
+        <xacro:property name="laser_calibration" value="${dict(xyz = [0, 0, 0], rpy = [0, 0, 0])}" />
+        <xacro:property name="camera_calibration" value="${dict(xyz = [0, 0, 0], rpy = [0, 0, 0])}" />
+    </xacro:unless>
+    <xacro:if value="$(arg calibrated)">
+        <xacro:property name="laser_calibration" value="${load_yaml('$(arg laser_calibration_file)')}" />
+        <xacro:property name="camera_calibration" value="${load_yaml('$(arg camera_calibration_file)')}" />
+    </xacro:if>
     <!-- main lemonbot macro -->
     <xacro:macro name="lemonbot" params="prefix">
@@ -34,5 +46,5 @@
         <!-- joint: ptu_mount_link to camera_mount -->
         <joint name="{prefix}_ptu_mount_link_to_camera_mount_link_joint" type="fixed">
-            <origin xyz="0.03 -0.1 0.1" rpy="-1.57 0 0" />
+            <origin xyz="${camera_calibration['xyz'][0]} ${camera_calibration['xyz'][1]} ${camera_calibration['xyz'][2]}" rpy="${camera_calibration['rpy'][0]} ${camera_calibration['rpy'][1]} ${camera_calibration['rpy'][2]}" />
             <parent link="${prefix}_ptu_mount_link" />
             <child link="${prefix}_camera_mount_link" />
@@ -40,5 +52,5 @@
         <!-- joint: ptu_mount_link to laser_optical_frame  -->
         <joint name="{prefix}_ptu_mount_link_to_laser_optical_frame" type="fixed">
-            <origin xyz="0 -0.05 0.1" rpy="1.57 -1.57 0" />
+            <origin xyz="${laser_calibration['xyz'][0]} ${laser_calibration['xyz'][1]} ${laser_calibration['xyz'][2]}" rpy="${laser_calibration['rpy'][0]} ${laser_calibration['rpy'][1]} ${laser_calibration['rpy'][2]}" />
             <parent link="${prefix}_ptu_mount_link" />
             <child link="${prefix}_laser_optical_frame" />

Commit message: a new version for lemonbot.

File: lemonbot_description/urdf/lemonbot.urdf.xacro (robot description, xacro)
@@ -2,8 +2,6 @@
 <robot
     xmlns:xacro="http://www.ros.org/wiki/xacro" name="lemonbot">
-    <xacro:arg name="calibrated" default="false"/>
-    <xacro:arg name="laser_calibration_file" default="$(find lemonbot_calibration)/calibration/camera_calibration.yaml" />
-    <xacro:arg name="camera_calibration_file" default="$(find lemonbot_calibration)/calibration/camera_calibration.yaml" />
     <xacro:include filename="$(find lemonbot_description)/urdf/lemonbot_macro.urdf.xacro"/>
-    <xacro:lemonbot prefix="lemonbot" />
+    <xacro:lemonbot prefix="lemonbot_">
+    </xacro:lemonbot>
 </robot>

File: lemonbot_description/urdf/lemonbot_macro.urdf.xacro (robot description, xacro)
@@ -1,62 +1,42 @@
 <?xml version="1.0"?>
 <robot xmlns:xacro="http://www.ros.org/wiki/xacro">
-  <xacro:arg name="calibrated" default="false"/>
-  <xacro:arg name="laser_calibration_file" default="" />
-  <xacro:arg name="camera_calibration_file" default="" />
-  <!-- include all the dependencies -->
-  <!-- include asus_camera macro from hector_sensors_description -->
-  <xacro:include filename="$(find hector_sensors_description)/urdf/asus_camera.urdf.xacro"/>
+  <!-- dependencies -->
   <!-- include ptu_d46 macro from flir_ptu_description -->
   <xacro:include filename="$(find flir_ptu_description)/urdf/d46.urdf.xacro" />
   <!-- include sick lms1xx macro from lms1xx -->
   <xacro:include filename="$(find lms1xx)/urdf/sick_lms1xx.urdf.xacro" />
-  <!-- load calibration -->
-  <xacro:unless value="$(arg calibrated)">
-    <xacro:property name="laser_calibration" value="${dict(xyz = [0, 0, 0], rpy = [0, 0, 0])}" />
-    <xacro:property name="camera_calibration" value="${dict(xyz = [0, 0, 0], rpy = [0, 0, 0])}" />
-  </xacro:unless>
-  <xacro:if value="$(arg calibrated)">
-    <xacro:property name="laser_calibration" value="${load_yaml('$(arg laser_calibration_file)')}" />
-    <xacro:property name="camera_calibration" value="${load_yaml('$(arg camera_calibration_file)')}" />
-  </xacro:if>
   <!-- main lemonbot macro -->
   <xacro:macro name="lemonbot" params="prefix">
     <!-- links -->
     <!-- link: lemonbot_base_link -->
-    <link name="${prefix}_base_link" />
+    <link name="${prefix}base_link" />
     <!-- link: lemonbot_camera_mount_link -->
-    <link name="${prefix}_camera_mount_link" />
+    <link name="${prefix}camera_mount_link" />
     <!-- macros -->
     <!-- macro: ptu_d46 -->
-    <xacro:ptu_d46 name="${prefix}_ptu" />
-    <!-- macro: asus_camera -->
-    <!-- <xacro:asus_camera name="${prefix}_camera" parent="${prefix}_camera_mount_link"><origin xyz="0 0 0" rpy="0 0 0" /></xacro:asus_camera> -->
+    <xacro:ptu_d46 name="${prefix}ptu" />
     <!-- macro: sick_lms1xx -->
-    <xacro:sick_lms1xx frame="${prefix}_laser_optical_frame" />
+    <xacro:sick_lms1xx frame="${prefix}laser_optical_frame" />
     <!-- joints -->
     <!-- joint: base_link to ptu_joint -->
-    <joint name="${prefix}_base_link_to_ptu_joint" type="fixed">
+    <joint name="${prefix}base_link_to_ptu_joint" type="fixed">
       <origin xyz="0 0 0" rpy="0 0 0" />
-      <parent link="${prefix}_base_link" />
-      <child link="${prefix}_ptu_base_link" />
+      <parent link="${prefix}base_link" />
+      <child link="${prefix}ptu_base_link" />
     </joint>
-    <!-- joint: ptu_mount_link to camera_mount -->
-    <joint name="{prefix}_ptu_mount_link_to_camera_mount_link_joint" type="fixed">
-      <origin xyz="${camera_calibration['xyz'][0]} ${camera_calibration['xyz'][1]} ${camera_calibration['xyz'][2]}" rpy="${camera_calibration['rpy'][0]} ${camera_calibration['rpy'][1]} ${camera_calibration['rpy'][2]}" />
-      <parent link="${prefix}_ptu_mount_link" />
-      <child link="${prefix}_camera_mount_link" />
+    <!-- joint: ptu_mount_link to camera_mount_link -->
+    <joint name="{prefix}_ptu_mount_link_to_${prefix}camera_mount_link_joint" type="fixed">
+      <origin xyz="0 0 0" rpy="0 0 0" />
+      <parent link="${prefix}ptu_mount_link" />
+      <child link="${prefix}camera_mount_link" />
     </joint>
-    <!-- <link name="${prefix}_laser_mount_frame" /> -->
     <!-- joint: ptu_mount_link to laser_optical_frame  -->
-    <joint name="{prefix}_camera_mount_link_to_laser_optical_frame" type="fixed">
-      <origin xyz="${laser_calibration  ['xyz'][0]} ${laser_calibration['xyz'][1]} ${laser_calibration['xyz'][2]}" rpy="${laser_calibration['rpy'][0]} ${laser_calibration['rpy'][1]} ${laser_calibration['rpy'][2]}" />
-      <parent link="${prefix}_camera_mount_link" />
-      <child link="${prefix}_laser_optical_frame" />
+    <joint name="{prefix}ptu_mount_link_to_{prefix}laser_optical_link_joint" type="fixed">
+      <origin
+        xyz="-0.00862729  0.11007474  0.08132132"
+        rpy="2.23239 -1.54198 -0.64552" />
+      <parent link="${prefix}ptu_mount_link" />
+      <child link="${prefix}laser_optical_frame" />
     </joint>
-    <!-- <joint name="{prefix}_laser_mount_frame_to_laser_optical_frame" type="fixed">
-      <origin xyz="0 0 0" rpy="${-pi/2} ${-pi/2} 0" />
-      <parent link="${prefix}_laser_mount_frame" />
-      <child link="${prefix}_laser_optical_frame" />
-    </joint> -->
   </xacro:macro>
 </robot>
