Commit message: some minor changes

File: lemonbot_description/urdf/lemonbot_macro.urdf.xacro (robot description, xacro)
@@ -1,59 +1,59 @@
 <?xml version="1.0"?>
 <robot
-    xmlns:xacro="http://www.ros.org/wiki/xacro">
-    <xacro:arg name="calibrated" default="false"/>
-    <xacro:arg name="laser_calibration_file" default="" />
-    <xacro:arg name="camera_calibration_file" default="" />
-    <!-- include all the dependencies -->
-    <!-- include asus_camera macro from hector_sensors_description -->
-    <xacro:include filename="$(find hector_sensors_description)/urdf/asus_camera.urdf.xacro"/>
-    <!-- include ptu_d46 macro from flir_ptu_description -->
-    <xacro:include filename="$(find flir_ptu_description)/urdf/d46.urdf.xacro" />
-    <!-- include sick lms1xx macro from lms1xx -->
-    <xacro:include filename="$(find lms1xx)/urdf/sick_lms1xx.urdf.xacro" />
-    <!-- load calibration -->
-    <xacro:unless value="$(arg calibrated)">
-        <xacro:property name="laser_calibration" value="${dict(xyz = [0, 0, 0], rpy = [0, 0, 0])}" />
-        <xacro:property name="camera_calibration" value="${dict(xyz = [0, 0, 0], rpy = [0, 0, 0])}" />
-    </xacro:unless>
-    <xacro:if value="$(arg calibrated)">
-        <xacro:property name="laser_calibration" value="${load_yaml('$(arg laser_calibration_file)')}" />
-        <xacro:property name="camera_calibration" value="${load_yaml('$(arg camera_calibration_file)')}" />
-    </xacro:if>
-    <!-- main lemonbot macro -->
-    <xacro:macro name="lemonbot" params="prefix">
-        <!-- links -->
-        <!-- link: lemonbot_base_link -->
-        <link name="${prefix}_base_link" />
-        <!-- link: lemonbot_camera_mount_link -->
-        <link name="${prefix}_camera_mount_link" />
-        <!-- macros -->
-        <!-- macro: ptu_d46 -->
-        <xacro:ptu_d46 name="${prefix}_ptu" />
-        <!-- macro: asus_camera -->
-        <xacro:asus_camera name="${prefix}_camera" parent="${prefix}_camera_mount_link">
-            <origin xyz="0 0 0" rpy="0 0 0" />
-        </xacro:asus_camera>
-        <!-- macro: sick_lms1xx -->
-        <xacro:sick_lms1xx frame="${prefix}_laser_optical_frame" />
-        <!-- joints -->
-        <!-- joint: base_link to ptu_joint -->
-        <joint name="${prefix}_base_link_to_ptu_joint" type="fixed">
-            <origin xyz="0 0 0" rpy="0 0 0" />
-            <parent link="${prefix}_base_link" />
-            <child link="${prefix}_ptu_base_link" />
-        </joint>
-        <!-- joint: ptu_mount_link to camera_mount -->
-        <joint name="{prefix}_ptu_mount_link_to_camera_mount_link_joint" type="fixed">
-            <origin xyz="${camera_calibration['xyz'][0]} ${camera_calibration['xyz'][1]} ${camera_calibration['xyz'][2]}" rpy="${camera_calibration['rpy'][0]} ${camera_calibration['rpy'][1]} ${camera_calibration['rpy'][2]}" />
-            <parent link="${prefix}_ptu_mount_link" />
-            <child link="${prefix}_camera_mount_link" />
-        </joint>
-        <!-- joint: ptu_mount_link to laser_optical_frame  -->
-        <joint name="{prefix}_ptu_mount_link_to_laser_optical_frame" type="fixed">
-            <origin xyz="${laser_calibration['xyz'][0]} ${laser_calibration['xyz'][1]} ${laser_calibration['xyz'][2]}" rpy="${laser_calibration['rpy'][0]} ${laser_calibration['rpy'][1]} ${laser_calibration['rpy'][2]}" />
-            <parent link="${prefix}_ptu_mount_link" />
-            <child link="${prefix}_laser_optical_frame" />
-        </joint>
-    </xacro:macro>
+  xmlns:xacro="http://www.ros.org/wiki/xacro">
+  <xacro:arg name="calibrated" default="false"/>
+  <xacro:arg name="laser_calibration_file" default="" />
+  <xacro:arg name="camera_calibration_file" default="" />
+  <!-- include all the dependencies -->
+  <!-- include asus_camera macro from hector_sensors_description -->
+  <xacro:include filename="$(find hector_sensors_description)/urdf/asus_camera.urdf.xacro"/>
+  <!-- include ptu_d46 macro from flir_ptu_description -->
+  <xacro:include filename="$(find flir_ptu_description)/urdf/d46.urdf.xacro" />
+  <!-- include sick lms1xx macro from lms1xx -->
+  <xacro:include filename="$(find lms1xx)/urdf/sick_lms1xx.urdf.xacro" />
+  <!-- load calibration -->
+  <xacro:unless value="$(arg calibrated)">
+    <xacro:property name="laser_calibration" value="${dict(xyz = [0, 0, 0], rpy = [0, 0, 0])}" />
+    <xacro:property name="camera_calibration" value="${dict(xyz = [0, 0, 0], rpy = [0, 0, 0])}" />
+  </xacro:unless>
+  <xacro:if value="$(arg calibrated)">
+    <xacro:property name="laser_calibration" value="${load_yaml('$(arg laser_calibration_file)')}" />
+    <xacro:property name="camera_calibration" value="${load_yaml('$(arg camera_calibration_file)')}" />
+  </xacro:if>
+  <!-- main lemonbot macro -->
+  <xacro:macro name="lemonbot" params="prefix">
+    <!-- links -->
+    <!-- link: lemonbot_base_link -->
+    <link name="${prefix}_base_link" />
+    <!-- link: lemonbot_camera_mount_link -->
+    <link name="${prefix}_camera_mount_link" />
+    <!-- macros -->
+    <!-- macro: ptu_d46 -->
+    <xacro:ptu_d46 name="${prefix}_ptu" />
+    <!-- macro: asus_camera -->
+    <xacro:asus_camera name="${prefix}_camera" parent="${prefix}_camera_mount_link">
+      <origin xyz="0 0 0" rpy="0 0 0" />
+    </xacro:asus_camera>
+    <!-- macro: sick_lms1xx -->
+    <xacro:sick_lms1xx frame="${prefix}_laser_optical_frame" />
+    <!-- joints -->
+    <!-- joint: base_link to ptu_joint -->
+    <joint name="${prefix}_base_link_to_ptu_joint" type="fixed">
+      <origin xyz="0 0 0" rpy="0 0 0" />
+      <parent link="${prefix}_base_link" />
+      <child link="${prefix}_ptu_base_link" />
+    </joint>
+    <!-- joint: ptu_mount_link to camera_mount -->
+    <joint name="{prefix}_ptu_mount_link_to_camera_mount_link_joint" type="fixed">
+      <origin xyz="${camera_calibration['xyz'][0]} ${camera_calibration['xyz'][1]} ${camera_calibration['xyz'][2]}" rpy="${camera_calibration['rpy'][0]} ${camera_calibration['rpy'][1]} ${camera_calibration['rpy'][2]}" />
+      <parent link="${prefix}_ptu_mount_link" />
+      <child link="${prefix}_camera_mount_link" />
+    </joint>
+    <!-- joint: ptu_mount_link to laser_optical_frame  -->
+    <joint name="{prefix}_ptu_mount_link_to_laser_optical_frame" type="fixed">
+      <origin xyz="${laser_calibration['xyz'][0]} ${laser_calibration['xyz'][1]} ${laser_calibration['xyz'][2]}" rpy="${laser_calibration['rpy'][0]} ${laser_calibration['rpy'][1]} ${laser_calibration['rpy'][2]}" />
+      <parent link="${prefix}_ptu_mount_link" />
+      <child link="${prefix}_laser_optical_frame" />
+    </joint>
+  </xacro:macro>
 </robot>

Commit message: first point cloud is done

File: lemonbot_description/urdf/lemonbot_macro.urdf.xacro (robot description, xacro)
@@ -32,7 +32,5 @@
     <xacro:ptu_d46 name="${prefix}_ptu" />
     <!-- macro: asus_camera -->
-    <xacro:asus_camera name="${prefix}_camera" parent="${prefix}_camera_mount_link">
-      <origin xyz="0 0 0" rpy="0 0 0" />
-    </xacro:asus_camera>
+    <!-- <xacro:asus_camera name="${prefix}_camera" parent="${prefix}_camera_mount_link"><origin xyz="0 0 0" rpy="0 0 0" /></xacro:asus_camera> -->
     <!-- macro: sick_lms1xx -->
     <xacro:sick_lms1xx frame="${prefix}_laser_optical_frame" />

Commit message: changed to parent of the laser to be the camera.

File: lemonbot_description/urdf/lemonbot_macro.urdf.xacro (robot description, xacro)
@@ -49,7 +49,7 @@
     </joint>
     <!-- joint: ptu_mount_link to laser_optical_frame  -->
-    <joint name="{prefix}_ptu_mount_link_to_laser_optical_frame" type="fixed">
+    <joint name="{prefix}_camera_mount_link_to_laser_optical_frame" type="fixed">
       <origin xyz="${laser_calibration['xyz'][0]} ${laser_calibration['xyz'][1]} ${laser_calibration['xyz'][2]}" rpy="${laser_calibration['rpy'][0]} ${laser_calibration['rpy'][1]} ${laser_calibration['rpy'][2]}" />
-      <parent link="${prefix}_ptu_mount_link" />
+      <parent link="${prefix}_camera_mount_link" />
       <child link="${prefix}_laser_optical_frame" />
     </joint>

Commit message: created node for automatic radlocc acquisition

File: lemonbot_description/urdf/lemonbot_macro.urdf.xacro (robot description, xacro)
@@ -50,5 +50,5 @@
     <!-- joint: ptu_mount_link to laser_optical_frame  -->
     <joint name="{prefix}_camera_mount_link_to_laser_optical_frame" type="fixed">
-      <origin xyz="${laser_calibration['xyz'][0]} ${laser_calibration['xyz'][1]} ${laser_calibration['xyz'][2]}" rpy="${laser_calibration['rpy'][0]} ${laser_calibration['rpy'][1]} ${laser_calibration['rpy'][2]}" />
+      <origin xyz="${laser_calibration  ['xyz'][0]} ${laser_calibration['xyz'][1]} ${laser_calibration['xyz'][2]}" rpy="${laser_calibration['rpy'][0]} ${laser_calibration['rpy'][1]} ${laser_calibration['rpy'][2]}" />
       <parent link="${prefix}_camera_mount_link" />
       <child link="${prefix}_laser_optical_frame" />

Commit message: managed to get a good calibration

File: lemonbot_description/urdf/lemonbot_macro.urdf.xacro (robot description, xacro)
@@ -1,5 +1,4 @@
 <?xml version="1.0"?>
-<robot
-  xmlns:xacro="http://www.ros.org/wiki/xacro">
+<robot xmlns:xacro="http://www.ros.org/wiki/xacro">
   <xacro:arg name="calibrated" default="false"/>
   <xacro:arg name="laser_calibration_file" default="" />
@@ -48,4 +47,5 @@
       <child link="${prefix}_camera_mount_link" />
     </joint>
+    <!-- <link name="${prefix}_laser_mount_frame" /> -->
     <!-- joint: ptu_mount_link to laser_optical_frame  -->
     <joint name="{prefix}_camera_mount_link_to_laser_optical_frame" type="fixed">
@@ -54,4 +54,9 @@
       <child link="${prefix}_laser_optical_frame" />
     </joint>
+    <!-- <joint name="{prefix}_laser_mount_frame_to_laser_optical_frame" type="fixed">
+      <origin xyz="0 0 0" rpy="${-pi/2} ${-pi/2} 0" />
+      <parent link="${prefix}_laser_mount_frame" />
+      <child link="${prefix}_laser_optical_frame" />
+    </joint> -->
   </xacro:macro>
 </robot>

Commit message: added exporter

File: lemonbot_description/urdf/lemonbot_macro.urdf.xacro (robot description, xacro)
@@ -17,5 +17,5 @@
     <xacro:ptu_d46 name="${prefix}ptu" />
     <!-- macro: sick_lms1xx -->
-    <xacro:sick_lms1xx frame="${prefix}laser_optical_frame" />
+    <xacro:sick_lms1xx frame="${prefix}laser_optical_link" />
     <!-- joints -->
     <!-- joint: base_link to ptu_joint -->
@@ -31,5 +31,5 @@
       <child link="${prefix}camera_mount_link" />
     </joint>
-    <!-- joint: ptu_mount_link to laser_optical_frame  -->
+    <!-- joint: ptu_mount_link to laser_optical_link  -->
     <joint name="{prefix}ptu_mount_link_to_{prefix}laser_optical_link_joint" type="fixed">
       <origin
@@ -37,5 +37,5 @@
         rpy="2.23239 -1.54198 -0.64552" />
       <parent link="${prefix}ptu_mount_link" />
-      <child link="${prefix}laser_optical_frame" />
+      <child link="${prefix}laser_optical_link" />
     </joint>
   </xacro:macro>
